Commit message: updated to accurate robot measurements

File: lrd_system/description/chassis.xacro (robot description, xacro)
@@ -5,14 +5,14 @@
     <!-- ROVER PROPERTIES -->
     <!-- mass in Kilograms, xyz in meters, rpy in radians -->
-    <xacro:property name="wheel_mass" value="2.019"/>
-    <xacro:property name="wheel_radius" value="0.194"/>
-    <xacro:property name="wheel_width" value="0.194"/>
-    <xacro:property name="wheel_dist_from_center" value="0.38735"/>
-    <xacro:property name="caster_wheel_mass" value="1.000"/>
-    <xacro:property name="caster_wheel_offset" value="0.725"/>
+    <xacro:property name="wheel_mass" value="0.0025"/>
+    <xacro:property name="wheel_radius" value="0.044"/>
+    <xacro:property name="wheel_width" value="0.01417"/>
+    <xacro:property name="wheel_dist_from_center" value="{0.125/2}"/>
+    <xacro:property name="caster_wheel_mass" value="0.0025"/>
+    <xacro:property name="caster_wheel_offset" value="0.135"/>
     <xacro:property name="chassis_mass" value="0.057"/>
-    <xacro:property name="chassis_width" value="0.566"/>
-    <xacro:property name="chassis_length" value="0.9398"/>
-    <xacro:property name="chassis_height" value="0.232"/>
+    <xacro:property name="chassis_width" value="0.105"/>
+    <xacro:property name="chassis_length" value="0.19"/>
+    <xacro:property name="chassis_height" value="0.0.065"/>
     <!-- BASE LINK -->
     <!-- Base link sits at bottom center of chassis -->

File: lrd_system/description/ros2_control.xacro (robot description, xacro)
@@ -1,6 +1,10 @@
 <?xml version="1.0"?>
 <robot xmlns:xacro="http://www.ros.org/wiki/xacro">
-    <!-- <xacro:property name="min_vel" value="-10"/>
-    <xacro:property name="max_vel" value="10"/> -->
+    <!--
+    Wheel radius = 0.044m
+    Max angular speed (rpm) = 175 rpm
+    Max angular speed (rad/s) = (175*pi/30)rad/s = 18.3259 rad/s
+    max linear speed (m/s) = (175*pi/30)*0.044 = 0.8063 m/s
+    -->
     <!-- hardware interface for controller manager -->
     <ros2_control name="GazeboSystem" type="system">
@@ -11,6 +15,6 @@
         <joint name="left_wheel_joint">
             <command_interface name="velocity">
-                <param name="min">-10</param>
-                <param name="max">10</param>
+                <param name="min">-18.3259</param>
+                <param name="max">18.3259</param>
             </command_interface>
             <state_interface name="velocity"/>
@@ -20,6 +24,6 @@
         <joint name="right_wheel_joint">
             <command_interface name="velocity">
-                <param name="min">-10</param>
-                <param name="max">10</param>
+                <param name="min">-18.3259</param>
+                <param name="max">18.3259</param>
             </command_interface>
             <state_interface name="velocity"/>

Commit message: slight improvements made to sim

File: lrd_system/description/chassis.xacro (robot description, xacro)
@@ -5,14 +5,14 @@
     <!-- ROVER PROPERTIES -->
     <!-- mass in Kilograms, xyz in meters, rpy in radians -->
-    <xacro:property name="wheel_mass" value="0.0025"/>
+    <xacro:property name="wheel_mass" value="0.030"/>
     <xacro:property name="wheel_radius" value="0.044"/>
     <xacro:property name="wheel_width" value="0.01417"/>
-    <xacro:property name="wheel_dist_from_center" value="{0.125/2}"/>
-    <xacro:property name="caster_wheel_mass" value="0.0025"/>
+    <xacro:property name="wheel_dist_from_center" value="${0.125/2 - 0.01417/2}"/>
+    <xacro:property name="caster_wheel_mass" value="0.002"/>
     <xacro:property name="caster_wheel_offset" value="0.135"/>
-    <xacro:property name="chassis_mass" value="0.057"/>
+    <xacro:property name="chassis_mass" value="0.660"/>
     <xacro:property name="chassis_width" value="0.105"/>
     <xacro:property name="chassis_length" value="0.19"/>
-    <xacro:property name="chassis_height" value="0.0.065"/>
+    <xacro:property name="chassis_height" value="0.065"/>
     <!-- BASE LINK -->
     <!-- Base link sits at bottom center of chassis -->

File: lrd_system/description/gazebo.xacro (robot description, xacro)
@@ -4,12 +4,19 @@
         <material>Gazebo/White</material>
     </gazebo>
+    <!-- mu used is for rubber on horseshoe-->
     <gazebo reference="left_wheel_link">
         <material>Gazebo/Blue</material>
+        <mu1 value="100.0"/>
+        <mu2 value="100.0"/>
     </gazebo>
     <gazebo reference="right_wheel_link">
         <material>Gazebo/Blue</material>
+        <mu1 value="100.0"/>
+        <mu2 value="100.0"/>
     </gazebo>
     <gazebo reference="caster_wheel_link">
         <material>Gazebo/Red</material>
+        <mu1 value="0.001"/>
+        <mu2 value="0.001"/>
     </gazebo>
     <!-- <gazebo reference="camera_pole_link">

File: lrd_system/description/ros2_control.xacro (robot description, xacro)
@@ -15,6 +15,6 @@
         <joint name="left_wheel_joint">
             <command_interface name="velocity">
-                <param name="min">-18.3259</param>
-                <param name="max">18.3259</param>
+                <param name="min">-10</param>
+                <param name="max">10</param>
             </command_interface>
             <state_interface name="velocity"/>
@@ -24,6 +24,6 @@
         <joint name="right_wheel_joint">
             <command_interface name="velocity">
-                <param name="min">-18.3259</param>
-                <param name="max">18.3259</param>
+                <param name="min">-10</param>
+                <param name="max">10</param>
             </command_interface>
             <state_interface name="velocity"/>
